File: mask-board.kicad_pcb (KiCad board)
At the start: 2 copper layers, 62.5 x 50.5 mm, 58 parts, among them J1 SWIM Connector, J2 I2C Breakout, M1 Fan_3pin, M2 Fan_3pin, M3 Motor_DC, Q1 2N7000, Q2 2N7000, Q3 2N7000, Q4 2N7000, SW1 SW_Push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

Commit message: Update to board V2
Parts:
- D1: footprint footprints:T2133BGR -> footprints:LED_T2133BGR
- moved J2 19.9 mm to (167.0, 115.6)
- moved J1 9.69 mm to (123.2, 108.0)
- moved R11 6.98 mm to (167.6, 105.4)
- moved D2 6.03 mm to (169.5, 99.4)
- moved M3 6.03 mm to (174.0, 98.1)
- moved Q2 6.03 mm to (172.4, 107.0)
- moved R10 6.03 mm to (165.1, 106.4)
- moved A1 5.72 mm to (123.2, 78.7)
- moved C17 1.08 mm to (165.6, 102.5)
- moved C18 1.08 mm to (161.8, 102.5)
- moved C19 1.08 mm to (163.7, 102.5)
Routing:
- net SWIM: track 43.5 -> 35.0 mm
- net RESET: track 34.1 -> 25.6 mm
- net +3V3: track 164.8 -> 157.4 mm
- net SCL: track 27.6 -> 33.9 mm
- net +5V: track 75.5 -> 71.3 mm
- net SDA: track 37.2 -> 35.0 mm
- net ERM_MOTOR: track 22.2 -> 20.1 mm
Other:
- board size 62.5 x 50.5 mm -> 56.5 x 41.9 mm
- board text added: "3V3"
- board text added: "5V"
- board text added: "BAT"
- board text added: "D+"
- board text added: "D-"
- board text added: "EN"
- board text added: "GND"
- board text added: "RESET"
- board text added: "SCL"
- board text added: "SDA"
- board text added: "SWIM"
- board text added: "VIN"
- board text added: "VU"
